File: Thermocoupe.sch (KiCad schematic (older format))
At the start: 0 parts

Commit message: Defining your inputs and outputs
Changed lines of the file:
@@
 Sheet 3 8
 Title ""
-Date "21 sep 2013"
+Date "26 sep 2013"
 Rev ""
 Comp ""
@@
 Text HLabel 8500 3450 2    60   Input ~ 0
 TC IN -
+Text HLabel 3600 2550 0    60   Input ~ 0
+MOSI
+Text HLabel 3600 2700 0    60   Output ~ 0
+MISO
+Text HLabel 3600 2850 0    60   Input ~ 0
+SCLK
+Text HLabel 3600 3000 0    60   Input ~ 0
+/CS
 $EndSCHEMATC

Commit message: Understanding the thermocouple module
Parts:
- added D?: ZENERSMALL, ~, symbol ZENERSMALL
- added R? (x7): R, ~, symbol R
- added U? (x4): LM324, symbol LM324
- added U? (x2): MCP3550-60-E/SN, SO8, symbol MCP3550-60-E/SN
Connections:
- net labels added: +12V, -12V, AGND
- wire segments 0 -> 45
Other:
- note added: "16-24Bit ADC"
- note added: "Analog/TC Input"
- note added: "General Temperature Sensor"
- note added: "Instrumentation Amp"
