File: Arduino.sch (KiCad schematic (older format))
At the start: 0 parts

Commit message: Arduino Module
Parts:
- added ARD?: ARDUINOPINS, symbol ARDUINOPINS
- added R? (x12): R, ~, symbol R
Connections:
- net MISO: now also R?.2
- net MOSI: now also R?.2
- net SCLK: now also R?.2
- new net: ARD?.11 (Digital0), R?.1
- new net: ARD?.12 (Digital1), R?.1
- new net: ARD?.18 (Digital7), R?.1
- new net: ARD?.19 (PWM0), R?.1
- new net: ARD?.20 (/CS), R?.1
- new net: ARD?.21 (MOSI), R?.1
- new net: ARD?.22 (MISO), R?.1
- new net: ARD?.23 (SCK), R?.1
- new net: ARD?.5 (Analog0), R?.2
- new net: ARD?.6 (Analog1), R?.2
- new net: ARD?.7 (Analog2), R?.2
- new net: ARD?.8 (Analog3), R?.2
- new net /CS_FAN: R?.2
- new net /CS_TC: R?.2
- new net /FAN_EN: R?.2
- new net CURR_MEAS: R?.1
- new net LED_EN_PWM: R?.2
- new net RELAY+: R?.2
- new net TACH_MEAS: R?.1
- new net V+_ADJ_MON: R?.1
- new net V-_ADJ_MON: R?.1
