File: Relay.sch (KiCad schematic (older format))
At the start: 0 parts

Commit message: Understanding the relay module
Parts:
- added D?: DIODE, ~, symbol DIODE
- added D?: LED, ~, symbol LED
- added K?: RELAY_SPDT, ~, symbol RELAY_SPDT
- added Q?: NPN, ~, symbol NPN
- added R? (x6): R, ~, symbol R
- added U?: PHTRANS, ~, symbol PHTRANS
Connections:
- net labels added: +12P, COM, GND, NC, NO
- net labels removed: Relay+, Relay-
- wire segments 0 -> 32
Changed lines of the file:
@@
 LIBS:contrib
 LIBS:valves
+LIBS:relay_spdt
 LIBS:CE-cache
 EELAYER 27 0
@@
 Comment4 ""
 $EndDescr
-Text HLabel 2300 2150 0    60   Input ~ 0
+Text HLabel 2500 3050 0    60   Input ~ 0
 DIN+
-Text HLabel 2300 2300 0    60   Input ~ 0
+Text HLabel 2500 3400 0    60   Input ~ 0
 DIN-
-Text HLabel 7700 2050 2    60   Input ~ 0
-Relay+
-Text HLabel 7700 2200 2    60   Output ~ 0
-Relay-
+Text HLabel 9350 2000 2    60   BiDi ~ 0
+NC
+Text HLabel 9350 2200 2    60   BiDi ~ 0
+NO
+$Comp
+L PHTRANS U?
+U 1 1 52444642
+P 4450 3250
+F 0 "U?" H 4400 3600 70  0000 C CNN
+F 1 "PHTRANS" H 4400 2900 70  0000 C CNN
+F 2 "~" H 4450 3250 60  0000 C CNN
+F 3 "~" H 4450 3250 60  0000 C CNN
+	1    4450 3250
+	1    0    0    -1
+$EndComp
+$Comp
+L R R?
+U 1 1 5244466F
+P 6450 3650
+F 0 "R?" H 6530 3650 40  0000 C CNN
+F 1 "R" V 6457 3651 40  0000 C CNN
+F 2 "~" V 6380 3650 30  0000 C CNN
+F 3 "~" H 6450 3650 30  0000 C CNN
+	1    6450 3650
+	0    -1   -1   0
+$EndComp
+$Comp
+L NPN Q?
+U 1 1 5244467E
+P 7400 3650
+F 0 "Q?" H 7400 3500 50  0000 R CNN
+F 1 "NPN" H 7400 3800 50  0000 R CNN
+F 2 "~" H 7400 3650 60  0000 C CNN
+F 3 "~" H 7400 3650 60  0000 C CNN
+	1    7400 3650
+	1    0    0    -1
+$EndComp
+$Comp
+L LED D?
+U 1 1 5244468D
+P 5400 4050
+F 0 "D?" H 5400 4150 50  0000 C CNN
+F 1 "LED" H 5400 3950 50  0000 C CNN
+F 2 "~" H 5400 4050 60  0000 C CNN
+F 3 "~" H 5400 4050 60  0000 C CNN
+	1    5400 4050
+	0    1    1    0
+$EndComp
+$Comp
+L RELAY_SPDT K?
+U 1 1 524435E1
+P 8750 2050
+F 0 "K?" H 8550 2300 70  0000 C CNN
+F 1 "RELAY_SPDT" H 8900 1550 70  0000 C CNN
+F 2 "~" H 8750 2050 60  0000 C CNN
+F 3 "~" H 8750 2050 60  0000 C CNN
+	1    8750 2050
+	1    0    0    -1
+$EndComp
+Text HLabel 9350 1500 2    60   BiDi ~ 0
+COM
+$Comp
+L R R?
+U 1 1 524438A5
+P 7500 4350
+F 0 "R?" H 7580 4350 40  0000 C CNN
+F 1 "R" V 7507 4351 40  0000 C CNN
+F 2 "~" V 7430 4350 30  0000 C CNN
+F 3 "~" H 7500 4350 30  0000 C CNN
+	1    7500 4350
+	-1   0    0    1
+$EndComp
+$Comp
+L GND #PWR?
+U 1 1 524438B5
+P 7500 5300
+F 0 "#PWR?" H 7500 5300 30  0001 C CNN
+F 1 "GND" H 7500 5230 30  0001 C CNN
+F 2 "" H 7500 5300 60  0000 C CNN
+F 3 "" H 7500 5300 60  0000 C CNN
+	1    7500 5300
+	1    0    0    -1
+$EndComp
+$Comp
+L R R?
+U 1 1 52443B2D
+P 5400 4600
+F 0 "R?" H 5480 4600 40  0000 C CNN
+F 1 "R" V 5407 4601 40  0000 C CNN
+F 2 "~" V 5330 4600 30  0000 C CNN
+F 3 "~" H 5400 4600 30  0000 C CNN
+	1    5400 4600
+	-1   0    0    1
+$EndComp
+Wire Wire Line
+	7900 2100 8350 2100
+Wire Wire Line
+	9150 2000 9350 2000
+Wire Wire Line
+	9150 2200 9350 2200
+Wire Wire Line
+	8350 2400 7500 2400
+Wire Wire Line
+	7500 2400 7500 3050
+Wire Wire Line
+	7500 3050 7500 3450
+Wire Wire Line
+	7200 3650 6700 3650
+Wire Wire Line
+	7500 3850 7500 4100
+Wire Wire Line
+	7500 4600 7500 4850
+Wire Wire Line
+	7500 4850 7500 5300
+Wire Wire Line
+	6450 2300 7000 2300
+Wire Wire Line
+	7000 2300 8350 2300
+Wire Wire Line
+	5400 4250 5400 4350
+Wire Wire Line
+	5400 3450 5400 3650
+Wire Wire Line
+	5400 3650 5400 3850
+Connection ~ 5400 3650
+$Comp
+L +12P #PWR?
+U 1 1 52443B6B
+P 6450 1500
+F 0 "#PWR?" H 6450 1470 30  0001 C CNN
+F 1 "+12P" H 6450 1600 30  0000 C CNN
+F 2 "" H 6450 1500 60  0000 C CNN
+F 3 "" H 6450 1500 60  0000 C CNN
+	1    6450 1500
+	1    0    0    -1
+$EndComp
+$Comp
+L R R?
+U 1 1 52443CC9
+P 3250 3400
+F 0 "R?" H 3330 3400 40  0000 C CNN
+F 1 "R" V 3257 3401 40  0000 C CNN
+F 2 "~" V 3180 3400 30  0000 C CNN
+F 3 "~" H 3250 3400 30  0000 C CNN
+	1    3250 3400
+	0    1    1    0
+$EndComp
+Wire Wire Line
+	3500 3400 3900 3400
+Wire Wire Line
+	2500 3050 3900 3050
+Wire Wire Line
+	2950 3400 2500 3400
+$Comp
+L R R?
+U 1 1 52443E35
+P 5500 3050
+F 0 "R?" H 5580 3050 40  0000 C CNN
+F 1 "R" V 5507 3051 40  0000 C CNN
+F 2 "~" V 5430 3050 30  0000 C CNN
+F 3 "~" H 5500 3050 30  0000 C CNN
+	1    5500 3050
+	0    -1   -1   0
+$EndComp
+Wire Wire Line
+	5000 3050 5250 3050
+Wire Wire Line
+	6450 3050 5750 3050
+Connection ~ 6450 2300
+Connection ~ 6450 3050
+Wire Wire Line
+	5400 4850 7500 4850
+Connection ~ 7500 4850
+$Comp
+L R R?
+U 1 1 524440F6
+P 6450 1900
+F 0 "R?" H 6530 1900 40  0000 C CNN
+F 1 "R" V 6457 1901 40  0000 C CNN
+F 2 "~" V 6380 1900 30  0000 C CNN
+F 3 "~" H 6450 1900 30  0000 C CNN
+	1    6450 1900
+	-1   0    0    1
+$EndComp
+Wire Wire Line
+	6450 1500 6450 1650
+Wire Wire Line
+	9350 1500 7900 1500
+Wire Wire Line
+	7900 1500 7900 2100
+$Comp
+L DIODE D?
+U 1 1 5244453B
+P 7000 2850
+F 0 "D?" H 7000 2950 40  0000 C CNN
+F 1 "DIODE" H 7000 2750 40  0000 C CNN
+F 2 "~" H 7000 2850 60  0000 C CNN
+F 3 "~" H 7000 2850 60  0000 C CNN
+	1    7000 2850
+	0    -1   -1   0
+$EndComp
+Wire Wire Line
+	7000 2650 7000 2300
+Connection ~ 7000 2300
+Wire Wire Line
+	6450 3250 5000 3250
+Wire Wire Line
+	6450 2150 6450 2300
+Wire Wire Line
+	6450 2300 6450 3050
+Wire Wire Line
+	6450 3050 6450 3250
+Wire Wire Line
+	7000 3050 7500 3050
+Connection ~ 7500 3050
+Wire Wire Line
+	5400 3650 6200 3650
+Wire Wire Line
+	5400 3450 5000 3450
 $EndSCHEMATC

Commit message: Arduino Module
Connections:
- net labels added: RELAY+, RELAY-, RELAY_COM, RELAY_NC, RELAY_NO
- net labels removed: COM, DIN+, DIN-, NC, NO
Changed lines of the file:
@@
 $EndDescr
 Text HLabel 2500 3050 0    60   Input ~ 0
-DIN+
+RELAY+
 Text HLabel 2500 3400 0    60   Input ~ 0
-DIN-
+RELAY-
 Text HLabel 9350 2000 2    60   BiDi ~ 0
-NC
+RELAY_NC
 Text HLabel 9350 2200 2    60   BiDi ~ 0
-NO
+RELAY_NO
 $Comp
 L PHTRANS U?
@@
 $EndComp
 Text HLabel 9350 1500 2    60   BiDi ~ 0
-COM
+RELAY_COM
 $Comp
 L R R?
